Commit message: neurons

File: body.urdf (robot description, URDF)
Before this commit: robot robot, 3 links, 2 joints
Links:
- removed link Backleg
- removed link Frontleg
- added link BackLeg, mass 1; collision box size=1 1 1; visual box size=1 1 1
- added link FrontLeg, mass 1; collision box size=1 1 1; visual box size=1 1 1
Joints:
- removed joint Torso_Frontleg
- added joint Torso_FrontLeg: type revolute, parent Torso, child FrontLeg, origin xyz=-0.5 0 1 rpy=0 0 0, axis 0 1 0, limit lower=-3.14159 upper=3.14159 effort=0.0 velocity=0.0
- joint Torso_BackLeg: child Backleg -> BackLeg

Commit message: hill-climber

File: body.urdf (robot description, URDF)
Before this commit: robot robot, 3 links, 2 joints
Joints:
- joint Torso_BackLeg: origin xyz=-0.5 0 1 rpy=0 0 0 -> xyz=0.5 0 1 rpy=0 0 0
- joint Torso_FrontLeg: origin xyz=0.5 0 1 rpy=0 0 0 -> xyz=-0.5 0 1 rpy=0 0 0

Commit message: quad

File: body.urdf (robot description, URDF)
Before this commit: robot robot, 3 links, 2 joints
Links:
- added link LeftLeg, mass 1; collision box size=1 0.2 0.2; visual box size=1 0.2 0.2
- added link LowerBackLeg, mass 1; collision box size=0.2 0.2 1; visual box size=0.2 0.2 1
- added link LowerFrontLeg, mass 1; collision box size=0.2 0.2 1; visual box size=0.2 0.2 1
- added link LowerLeftLeg, mass 1; collision box size=0.2 0.2 1; visual box size=0.2 0.2 1
- added link LowerRightLeg, mass 1; collision box size=0.2 0.2 1; visual box size=0.2 0.2 1
- added link RightLeg, mass 1; collision box size=1 0.2 0.2; visual box size=1 0.2 0.2
- link BackLeg: geometry collision box size=0.2 1 0.2; visual box size=0.2 1 0.2
- link FrontLeg: geometry collision box size=0.2 1 0.2; visual box size=0.2 1 0.2
Joints:
- added joint BackLeg_LowerBackLeg: type revolute, parent BackLeg, child LowerBackLeg, origin xyz=0 -1 0 rpy=0 0 0, axis 0 1 1, limit lower=-3.14159 upper=3.14159 effort=0.0 velocity=0.0
- added joint FrontLeg_LowerFrontLeg: type revolute, parent FrontLeg, child LowerFrontLeg, origin xyz=0 1 0 rpy=0 0 0, axis 0 1 1, limit lower=-3.14159 upper=3.14159 effort=0.0 velocity=0.0
- added joint LeftLeg_LowerLeftLeg: type revolute, parent LeftLeg, child LowerLeftLeg, origin xyz=-1 0 0 rpy=0 0 0, axis 0 1 1, limit lower=-3.14159 upper=3.14159 effort=0.0 velocity=0.0
- added joint RightLeg_LowerRightLeg: type revolute, parent RightLeg, child LowerRightLeg, origin xyz=1 0 0 rpy=0 0 0, axis 0 1 1, limit lower=-3.14159 upper=3.14159 effort=0.0 velocity=0.0
- added joint Torso_LeftLeg: type revolute, parent Torso, child LeftLeg, origin xyz=-0.5 0 1 rpy=0 0 0, axis 0 1 0, limit lower=-3.14159 upper=3.14159 effort=0.0 velocity=0.0
- added joint Torso_RightLeg: type revolute, parent Torso, child RightLeg, origin xyz=0.5 0 1 rpy=0 0 0, axis 0 1 0, limit lower=-3.14159 upper=3.14159 effort=0.0 velocity=0.0
- joint Torso_BackLeg: axis 0 1 0 -> 1 0 0; origin xyz=0.5 0 1 rpy=0 0 0 -> xyz=0 -0.5 1 rpy=0 0 0
- joint Torso_FrontLeg: axis 0 1 0 -> 1 0 0; origin xyz=-0.5 0 1 rpy=0 0 0 -> xyz=0 0.5 1 rpy=0 0 0

Commit message: snake finished

File: body.urdf (robot description, URDF)
Before this commit: robot robot, 9 links, 8 joints
Links:
- removed link BackLeg
- removed link FrontLeg
- removed link LeftLeg
- removed link LowerBackLeg
- removed link LowerFrontLeg
- removed link LowerLeftLeg
- removed link LowerRightLeg
- removed link RightLeg
- removed link Torso
- added link Cube0, mass 1; collision box size=1 1 1; visual box size=1 1 1
- added link Cube1, mass 1; collision box size=1 1 1; visual box size=1 1 1
- added link Cube2, mass 1; collision box size=1.2987677023572899 1.240726454272439 0.7112730979612141; visual box size=1.2987677023572899 1.240726454272439 0.7112730979612141
- added link Cube3, mass 1; collision box size=0.8010418801224821 0.9183287587396363 0.31871570975598135; visual box size=0.8010418801224821 0.9183287587396363 0.31871570975598135
- added link Cube4, mass 1; collision box size=0.9973186136484216 1.1426423193874646 1.1511879738988233; visual box size=0.9973186136484216 1.1426423193874646 1.1511879738988233
- added link Cube5, mass 1; collision box size=1.1473205875042873 0.4231604618861046 0.43741640046826585; visual box size=1.1473205875042873 0.4231604618861046 0.43741640046826585
- added link Cube6, mass 1; collision box size=1.2578273840169725 0.41634511601062413 0.6515129614460291; visual box size=1.2578273840169725 0.41634511601062413 0.6515129614460291
- added link Cube7, mass 1; collision box size=1.1841134522953773 0.37405762591125663 0.9423598266097608; visual box size=1.1841134522953773 0.37405762591125663 0.9423598266097608
Joints:
- removed joint BackLeg_LowerBackLeg
- removed joint FrontLeg_LowerFrontLeg
- removed joint LeftLeg_LowerLeftLeg
- removed joint RightLeg_LowerRightLeg
- removed joint Torso_BackLeg
- removed joint Torso_FrontLeg
- removed joint Torso_LeftLeg
- removed joint Torso_RightLeg
- added joint Cube0_Cube1: type revolute, parent Cube0, child Cube1, origin xyz=0 0.5 1 rpy=0 0 0, axis 1 0 1, limit lower=-3.14159 upper=3.14159 effort=0.0 velocity=0.0
- added joint Cube1_Cube2: type revolute, parent Cube1, child Cube2, origin xyz=0 1.1 0 rpy=0 0 0, axis 1 0 1, limit lower=-3.14159 upper=3.14159 effort=0.0 velocity=0.0
- added joint Cube2_Cube3: type revolute, parent Cube2, child Cube3, origin xyz=0 1.340726454272439 0 rpy=0 0 0, axis 1 0 1, limit lower=-3.14159 upper=3.14159 effort=0.0 velocity=0.0
- added joint Cube3_Cube4: type revolute, parent Cube3, child Cube4, origin xyz=0 1.0183287587396364 0 rpy=0 0 0, axis 1 0 1, limit lower=-3.14159 upper=3.14159 effort=0.0 velocity=0.0
- added joint Cube4_Cube5: type revolute, parent Cube4, child Cube5, origin xyz=0 1.2426423193874647 0 rpy=0 0 0, axis 1 0 1, limit lower=-3.14159 upper=3.14159 effort=0.0 velocity=0.0
- added joint Cube5_Cube6: type revolute, parent Cube5, child Cube6, origin xyz=0 0.5231604618861047 0 rpy=0 0 0, axis 1 0 1, limit lower=-3.14159 upper=3.14159 effort=0.0 velocity=0.0
- added joint Cube6_Cube7: type revolute, parent Cube6, child Cube7, origin xyz=0 0.5163451160106242 0 rpy=0 0 0, axis 1 0 1, limit lower=-3.14159 upper=3.14159 effort=0.0 velocity=0.0

Commit message: 3d

File: body.urdf (robot description, URDF)
Before this commit: robot robot, 8 links, 7 joints
Links:
- added link Cube10, mass 1; collision box size=1 1 0.5742109644213953; visual box size=1 1 0.5742109644213953
- added link Cube11, mass 1; collision box size=1 1 0.2663365135053904; visual box size=1 1 0.2663365135053904
- added link Cube12, mass 1; collision box size=1 0.6612972333066223 0.7759176353399244; visual box size=1 0.6612972333066223 0.7759176353399244
- added link Cube13, mass 1; collision box size=1 1 1; visual box size=1 1 1
- added link Cube14, mass 1; collision box size=1 0.7664974758359846 0.8266957140733586; visual box size=1 0.7664974758359846 0.8266957140733586
- added link Cube8, mass 1; collision box size=1 0.887352491677982 0.8196223106716563; visual box size=1 0.887352491677982 0.8196223106716563
- added link Cube9, mass 1; collision box size=1 0.8807879769642255 0.9207314931462072; visual box size=1 0.8807879769642255 0.9207314931462072
- link Cube2: geometry collision box size=1 0.49984787992978447 0.5615950007309369; visual box size=1 0.49984787992978447 0.5615950007309369
- link Cube3: geometry collision box size=1 0.26826264939607364 0.9219323462482565; visual box size=1 0.26826264939607364 0.9219323462482565
- link Cube4: geometry collision box size=1 0.6198772516392068 1; visual box size=1 0.6198772516392068 1
- link Cube5: geometry collision box size=1 0.3797110997496503 0.8674486066128253; visual box size=1 0.3797110997496503 0.8674486066128253
- link Cube6: geometry collision box size=1 1 0.572880593542435; visual box size=1 1 0.572880593542435
- link Cube7: geometry collision box size=1 0.6955167826089437 0.4091271808110037; visual box size=1 0.6955167826089437 0.4091271808110037
Joints:
- removed joint Cube1_Cube2
- removed joint Cube2_Cube3
- added joint Cube0_Cube2: type revolute, parent Cube0, child Cube2, origin xyz=0 -0.5 0 rpy=0 0 0, axis 0 0 1, limit lower=-3.14159 upper=3.14159 effort=0.0 velocity=0.0
- added joint Cube10_Cube12: type revolute, parent Cube10, child Cube12, origin xyz=-0.5 0.5 0 rpy=0 0 0, axis 0 0 1, limit lower=-3.14159 upper=3.14159 effort=0.0 velocity=0.0
- added joint Cube11_Cube14: type revolute, parent Cube11, child Cube14, origin xyz=-0.5 0 -0.1331682567526952 rpy=0 0 0, axis 1 0 0, limit lower=-3.14159 upper=3.14159 effort=0.0 velocity=0.0
- added joint Cube12_Cube13: type revolute, parent Cube12, child Cube13, origin xyz=-0.5 -0.33064861665331113 0 rpy=0 0 0, axis 0 0 1, limit lower=-3.14159 upper=3.14159 effort=0.0 velocity=0.0
- added joint Cube1_Cube3: type revolute, parent Cube1, child Cube3, origin xyz=-0.5 -0.5 0 rpy=0 0 0, axis 0 0 1, limit lower=-3.14159 upper=3.14159 effort=0.0 velocity=0.0
- added joint Cube7_Cube8: type revolute, parent Cube7, child Cube8, origin xyz=-0.5 0.34775839130447184 0 rpy=0 0 0, axis 0 0 1, limit lower=-3.14159 upper=3.14159 effort=0.0 velocity=0.0
- added joint Cube7_Cube9: type revolute, parent Cube7, child Cube9, origin xyz=-0.5 0 -0.20456359040550184 rpy=0 0 0, axis 1 0 0, limit lower=-3.14159 upper=3.14159 effort=0.0 velocity=0.0
- added joint Cube8_Cube10: type revolute, parent Cube8, child Cube10, origin xyz=-0.5 -0.443676245838991 0 rpy=0 0 0, axis 0 0 1, limit lower=-3.14159 upper=3.14159 effort=0.0 velocity=0.0
- added joint Cube9_Cube11: type revolute, parent Cube9, child Cube11, origin xyz=-0.5 0 0.4603657465731036 rpy=0 0 0, axis 1 0 0, limit lower=-3.14159 upper=3.14159 effort=0.0 velocity=0.0
- joint Cube0_Cube1: axis 1 0 1 -> 0 0 1; origin xyz=0 0.5 1 rpy=0 0 0 -> xyz=-0.5 0 0 rpy=0 0 0
- joint Cube3_Cube4: axis 1 0 1 -> 0 0 1; origin xyz=0 1.0183287587396364 0 rpy=0 0 0 -> xyz=-0.5 0.13413132469803682 0 rpy=0 0 0
- joint Cube4_Cube5: axis 1 0 1 -> 0 0 1; origin xyz=0 1.2426423193874647 0 rpy=0 0 0 -> xyz=-0.5 -0.3099386258196034 0 rpy=0 0 0
- joint Cube5_Cube6: axis 1 0 1 -> 0 0 1; origin xyz=0 0.5231604618861047 0 rpy=0 0 0 -> xyz=-0.5 0.18985554987482514 0 rpy=0 0 0
- joint Cube6_Cube7: axis 1 0 1 -> 0 0 1; origin xyz=0 0.5163451160106242 0 rpy=0 0 0 -> xyz=-0.5 -0.5 0 rpy=0 0 0
